File: hardware/pcbgalapagos.kicad_sch (KiCad schematic)
At the start: 51 parts, among them J1 Battery, U1 ESP32_DevKit, U2 INA226, U3 BME280, U4 LSM6DS, U5 MAX31855, U6 RFM95_Emissor, U7 GPS_NEO, U8 TPS62160DGK, U9 TPS62160DGK

Commit message: Final PCB, schematic and project libraries
Replace hardware with the final KiCad 10 project: module headers matched
to the real breakouts, GPS UART header, input protection, MISO series
termination, test points, solid SMD pour connections. Add the project
footprint library and fp-lib-table. Drop the outdated BOM and renders.
Parts:
- removed C11: 100nF 50V X7R, Capacitor_SMD:C_0805_2012Metric, symbol Device:C
- removed C12: 10uF 16V X7R, Capacitor_SMD:C_0805_2012Metric, symbol Device:C
- added D2: SMBJ13CA, Diode_SMD:D_SMB, symbol galapagos:D_TVS_Bidir
- added F1: MF-MSMF150/16X-2, Fuse:Fuse_1812_4532Metric, symbol galapagos:Polyfuse
- added Q11: DMP3056L-7, Package_TO_SOT_SMD:SOT-23, symbol galapagos:Q_PMOS_GSD
- added R9: 33, Resistor_SMD:R_0805_2012Metric, symbol Device:R
- added TP1, TP2, TP3, TP4: TestPoint, TestPoint:TestPoint_Pad_D1.5mm, symbol Connector:TestPoint
- added U10: GPS_NEO8M_UART, galapagos_fp:GPS_NEO8M_UART_Header_1x04, symbol galapagos:GPS_UART_Module
- C17, C19: value 10uF 25V X7R -> 10uF 50V X7R; footprint Capacitor_SMD:C_1206_3216Metric -> Capacitor_SMD:C_1210_3225Metric
- U1: footprint ESP32_Custom:ESP32_38Pin -> galapagos_fp:ESP32_DevKitC_V4_38
- U2: value INA226 -> INA260; footprint Connector_PinHeader_2.54mm:PinHeader_1x04_P2.54mm_Vertical -> galapagos_fp:Adafruit_INA260_Header; symbol galapagos:I2C_Module_4p -> galapagos:INA260_Module
- U3: footprint Connector_PinHeader_2.54mm:PinHeader_1x04_P2.54mm_Vertical -> galapagos_fp:Adafruit_BME280_Header; symbol galapagos:I2C_Module_4p -> galapagos:BME280_Module
- U4: value LSM6DS -> LSM6DSOX; footprint Connector_PinHeader_2.54mm:PinHeader_1x04_P2.54mm_Vertical -> galapagos_fp:Adafruit_LSM6DSOX_Header; symbol galapagos:I2C_Module_4p -> galapagos:LSM6DSOX_Module
- U5: footprint Connector_PinHeader_2.54mm:PinHeader_1x05_P2.54mm_Vertical -> galapagos_fp:Adafruit_MAX31855_Header; symbol galapagos:MAX31855_Module -> galapagos:MAX31855_Module6
- U6: footprint Connector_PinHeader_2.54mm:PinHeader_1x08_P2.54mm_Vertical -> galapagos_fp:RFM9x_Breakout_attexx; symbol galapagos:RFM95_Module -> galapagos:RFM9x_Breakout
- U7: footprint Connector_PinHeader_2.54mm:PinHeader_1x04_P2.54mm_Vertical -> galapagos_fp:GPS_I2C_Header_1x04
Connections:
- net +3V3: now also TP2.1
- net +3V3_GPS: now also U10.1 (VCC)
- net +3V3_RF: now also U6.11 (3V3); no longer U6.8 (3V3)
- net +5V: now also MOD1.2 (VCC), TP3.1; no longer MOD1.1 (5V), U1.19 (5V)
- net GND: now also MOD1.1 (GND), U3.3 (GND), U4.3 (GND), U5.3 (GND), D2.2 (A2), Q11.1 (G), TP4.1, U10.4 (GND); no longer MOD1.2 (GND), U3.2 (GND), U4.2 (GND), U5.2 (GND)
- net HSPI_MISO: now also R9.1; no longer MOD1.3 (MISO)
- net I2C_SCL: now also U3.4 (SCK), U4.4 (SCL); no longer U3.3 (SCL), U4.3 (SCL)
- net I2C_SDA: now also U3.6 (SDI), U4.5 (SDA); no longer U3.4 (SDA), U4.4 (SDA)
- net MAX_CLK: now also U5.6 (CLK); no longer U5.5 (CLK)
- net MAX_CS: now also U5.5 (CS); no longer U5.4 (CS)
- net MAX_DO: now also U1.5 (IO34), U5.4 (DO); no longer U1.13 (IO12), U5.3 (DO)
- net RFM_DIO0: now also U6.10 (DIO0); no longer U6.6 (DIO0)
- net RFM_RST: now also U6.6 (RST); no longer U6.7 (RST)
- net VBAT: now also Q11.2 (S), TP1.1; no longer J1.1 (Pin_1)
- net RFM_DIO1: now reaches U1.10 (IO26)
- net RFM_DIO1: now also U6.9 (DIO1)
- net GPS_TXD: now reaches U1.6 (IO35)
- net GPS_TXD: now also U10.3 (TX)
- net GPS_RXD: now reaches U1.7 (IO32)
- net GPS_RXD: now also U10.2 (RX)
- new net HSPI_MISO_SD: MOD1.3 (MISO), R9.2
- new net VBAT_F: D2.1 (A1), F1.2, Q11.3 (D)
- new net VBAT_IN: F1.1, J1.1 (Pin_1)
- no-connect marks 20 -> 36
Other:
- note added: "Battery: 3S3P Li-ion, 9.0 to 12.6 V (5 V rail needs Vin > 5.5 V, TPS62160 max 17 V)"
- note added: "ESP32 5V pin not connected: the DevKit is powered from +3V3 (U8) through its 3V3 pin. MAX_DO on IO34 (input only) instead of the IO12 strapping pin."
- note added: "GPS: solder only one header (U7 I2C or U10 UART)"
- note added: "INPUT PROTECTION (3S Li-ion)"
- note added: "PTC 1.5 A hold, TVS 13 V standoff, P-FET reverse-polarity switch (VGS max 25 V)"
- note added: "R9 sits at MOD1 pin 3 (MISO source)"
- note added: "TEST POINTS"
- note added: "at MOD1 pin 1 (+5V)"
- note added: "at U6 pin 8 (+3V3_RF)"
- note removed: "Battery: 6-8x Energizer L91 in series (5 V rail needs Vin > 5.5 V, max 17 V)"
- note removed: "U6 RFM95"
- moved on the sheet: C1, C10, C13, C14, C15, C16, C2, C22, C24, C25, C3, C4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
