File: hardware/pcbgalapagos.kicad_pcb (KiCad board)
At the start: 2 copper layers, 140.5 x 106 mm, 62 parts, among them J1 Battery, Q11 DMP3056L-7, U1 ESP32_DevKit, U10 GPS_NEO8M_UART, U2 INA260, U3 BME280, U4 LSM6DSOX, U5 MAX31855, U6 RFM95_Emissor, U7 GPS_NEO, U8 TPS62160DGK, U9 TPS62160DGK

Commit message: PCB: move parts under the modules to the bottom side
Decoupling caps C1-C6, C15, ferrites FB3/FB4 and SPI terminations R1/R2
now sit on the bottom layer next to the module header pins, so nothing
is sandwiched between the board and the plug-in modules.
Parts:
- C1, C15, C2, C3, C4, C5, C6, FB3, FB4, R1, R2: moved to B.Cu
- moved C6 3.72 mm to (121.0, 92.2)
- moved C2 3.71 mm to (118.5, 72.4)
- moved C4 3.67 mm to (97.6, 65.7)
- moved C5 3.20 mm to (121.0, 90.2)
- moved C1 3.20 mm to (118.5, 70.4)
- moved FB3 2.95 mm to (93.5, 56.5)
- moved C3 2.90 mm to (97.6, 63.7)
- moved FB4 1.60 mm to (206.0, 62.8)
- moved C15 1.28 mm to (207.4, 66.4), turned to 180 degrees
Routing:
- net HSPI_SCK: track 57.6 -> 70.2 mm, vias 0 -> 1
- net +3V3: track 285.0 -> 295.3 mm, vias 0 -> 2
- net HSPI_MOSI: track 52.5 -> 62.6 mm, vias 0 -> 1
- net +3V3_GPS: track 20.9 -> 13.2 mm
- net GND: track 47.1 -> 39.6 mm, vias 121 -> 123
- net HSPI_SCK_MCU: track 3.52 -> 7.04 mm
- net HSPI_MOSI_MCU: track 3.52 -> 7.04 mm
- net +3V3_RF: track 8.44 -> 10.2 mm
